Commit message: added pybullet ik

File: baxter_gym/robot_info/baxter/baxter_description/urdf/baxter_mod.urdf (robot description, URDF)
Before this commit: robot baxter, 49 links, 48 joints
Joints:
- joint left_endpoint: origin xyz=0.0 0 0.025 rpy=0 0 0 -> xyz=0.0 0 0.1327 rpy=0 0 0
- joint right_endpoint: origin xyz=0.0 0 0.025 rpy=0 0 0 -> xyz=0.0 0 0.1327 rpy=0 0 0
